Commit message: Updated Marrtino mass

File: marrtino_description/urdf/marrtino_robot.xacro (robot description, xacro)
@@ -48,5 +48,5 @@
 			<origin xyz="0 0 ${base_z_size/2}" rpy = "0 0 0" />
 		</collision>
-		<xacro:default_inertial mass="10"/>
+		<xacro:default_inertial mass="5"/>
 	</link>
 	<link name="left_wheel_link">
@@ -66,5 +66,5 @@
 			<origin xyz="0 0 0" rpy="${M_PI/2} 0 0"/>
 		</collision>
-		<xacro:default_inertial mass="1"/>
+		<xacro:default_inertial mass="0.5"/>
 	</link>
 	<link name="right_wheel_link">
@@ -84,5 +84,5 @@
 			<origin xyz="0 0 0" rpy="${M_PI/2} 0 0"/>
 		</collision>
-		<xacro:default_inertial mass="1"/>
+		<xacro:default_inertial mass="0.5"/>
 	</link>
 	<link name="block" type="fixed">
@@ -102,5 +102,5 @@
 			<origin xyz="0 0 -0.05" rpy = "0 0 0"/>
 		</collision>
-		<xacro:default_inertial mass="1"/>
+		<xacro:default_inertial mass="0.1"/>
 	</link>
 	<link name="castor_link">
@@ -120,5 +120,5 @@
 			<origin rpy="${M_PI/2} 0 0" xyz="0 0 0"/>
 		</collision>
-		<xacro:default_inertial mass="1"/>
+		<xacro:default_inertial mass="0.25"/>
 	</link>
 	<!-- Hokuyo Laser -->
@@ -136,10 +136,5 @@
 			</geometry>
 		</collision>
-		<inertial>
-			<mass value="1e-5"/>
-			<origin rpy="0 0 0" xyz="0 0 0"/>
-			<inertia ixx="1e-6" ixy="0" ixz="0"
-				 iyy="1e-6" iyz="0" izz="1e-6"/>
-		</inertial>
+		<xacro:default_inertial mass="0.1"/>
 	</link>
 <!-- ..........................................Joints definitions .....................................................-->

Commit message: Updated inertia parameters

File: marrtino_description/urdf/marrtino_robot.xacro (robot description, xacro)
@@ -30,4 +30,28 @@
 		</inertial>
 	</xacro:macro>
+	<xacro:macro name="cylinder_inertia" params="m r h">
+		<inertial>
+		<mass value="${m}" />
+	     <inertia  ixx="${m*(3*r*r+h*h)/12}" ixy = "0" ixz = "0"
+	                  iyy="${m*(3*r*r+h*h)/12}" iyz = "0"
+	                  izz="${m*r*r/2}" />
+		</inertial>
+	</xacro:macro>
+	<xacro:macro name="box_inertia" params="m x y z">
+		<inertial>
+		<mass value="${m}" />
+	        <inertia  ixx="${m*(y*y+z*z)/12}" ixy = "0" ixz = "0"
+	                  iyy="${m*(x*x+z*z)/12}" iyz = "0"
+	                  izz="${m*(x*x+z*z)/12}" />
+				</inertial>
+	</xacro:macro>
+	<xacro:macro name="sphere_inertia" params="m r">
+		<inertial>
+		<mass value="${m}" />
+	        <inertia  ixx="${2*m*r*r/5}" ixy = "0" ixz = "0"
+	                  iyy="${2*m*r*r/5}" iyz = "0"
+	                  izz="${2*m*r*r/5}" />
+	  </inertial>
+	</xacro:macro>
 <!-- ..........................................Links definitions .....................................................-->
 	<link name="base_footprint"/>
@@ -48,5 +72,5 @@
 			<origin xyz="0 0 ${base_z_size/2}" rpy = "0 0 0" />
 		</collision>
-		<xacro:default_inertial mass="5"/>
+		<xacro:box_inertia m="5" x="${base_x_size}" y="${base_y_size}" z="${base_z_size}"/>
 	</link>
 	<link name="left_wheel_link">
@@ -66,5 +90,5 @@
 			<origin xyz="0 0 0" rpy="${M_PI/2} 0 0"/>
 		</collision>
-		<xacro:default_inertial mass="0.5"/>
+		<xacro:cylinder_inertia m="0.5" r="${wheel_radius}" h="${wheel_lenght}" />
 	</link>
 	<link name="right_wheel_link">
@@ -84,12 +108,12 @@
 			<origin xyz="0 0 0" rpy="${M_PI/2} 0 0"/>
 		</collision>
-		<xacro:default_inertial mass="0.5"/>
+		<xacro:cylinder_inertia m="0.5" r="${wheel_radius}" h="${wheel_lenght}" />
 	</link>
 	<link name="block" type="fixed">
 		<visual>
 			<geometry>
-				<box size="0.03 0.03 0.10"/>
-			</geometry>
-			<origin xyz="0 0 -0.05" rpy = "0 0 0"/>
+				<box size="0.03 0.03 0.05"/>
+			</geometry>
+			<origin xyz="0 0 -0.025" rpy = "0 0 0"/>
 			<material name="red">
 				<color rgba="1 0 0 1"/>
@@ -98,9 +122,9 @@
 		<collision>
 			<geometry>
-				<box size="0.03 0.03 0.10"/>
+				<box size="0.03 0.03 0.05"/>
 			</geometry>
 			<origin xyz="0 0 -0.05" rpy = "0 0 0"/>
 		</collision>
-		<xacro:default_inertial mass="0.1"/>
+		<xacro:box_inertia m="0.05" x="0.03" y="0.03" z="0.05" />
 	</link>
 	<link name="castor_link">
@@ -119,9 +143,20 @@
 			</geometry>
 			<origin rpy="${M_PI/2} 0 0" xyz="0 0 0"/>
-		</collision>
-		<xacro:default_inertial mass="0.25"/>
+			<surface>
+        <friction>
+          <ode>
+            <mu>0</mu>
+            <mu2>0</mu2>
+            <slip1>1.0</slip1>
+            <slip2>1.0</slip2>
+          </ode>
+        </friction>
+			</surface>
+		</collision>
+		<xacro:cylinder_inertia m="0.25" r="${castor_radius}" h="${castor_length}" />
 	</link>
 	<!-- Hokuyo Laser -->
-	<link name="laser" >
+	<!--
+	<link name="laser_link" >
 		<visual>
 			<origin xyz="0 0 0" rpy="0 0 0"/>
@@ -136,5 +171,24 @@
 			</geometry>
 		</collision>
-		<xacro:default_inertial mass="0.1"/>
+		<xacro:box_inertia m="0.05" x="0.1" y="0.1" z="0.1" />
+	</link>
+-->
+	<link name="laser_link" >
+		<visual>
+			<origin xyz="0 0 0" rpy="0 0 0"/>
+			<geometry>
+				<cylinder length="0.03" radius="0.04"/>
+			</geometry>
+			<material name="black">
+				<color rgba="0 0 0 1"/>
+			</material>
+		</visual>
+		<collision>
+			<origin rpy="0 0 0" xyz="0 0 0"/>
+			<geometry>
+				<cylinder length="0.03" radius="0.04"/>
+			</geometry>
+		</collision>
+		<xacro:cylinder_inertia m="0.05" r="0.04" h="0.03" />
 	</link>
 <!-- ..........................................Joints definitions .....................................................-->
@@ -151,8 +205,8 @@
 		<axis xyz="0 1 0" />
 	</joint>
-	<joint name="castor_joint" type="continuous">
+	<joint name="castor_joint" type="fixed">
 		<parent link="block" />
 		<child link="castor_link" />
-		<origin xyz="0 0 -0.085" rpy="0 0 0"/>-->
+		<origin xyz="0 0 -0.065" rpy="0 0 0"/>-->
 		<axis xyz="0 1 0" />
 	</joint>
@@ -166,12 +220,12 @@
 		<parent link="base_footprint" />
 		<child link="base_link" />
-		<origin xyz="0.0 0.0 ${wheel_radius + 0.03}" rpy="0 0 ${M_PI}"/>
+		<origin xyz="0.0 0.0 ${wheel_radius + 0.03}" rpy="0 0 0"/>
 		<axis xyz="0 1 0" />
 	</joint>
 	<!--  Laser joint -->
-	<joint name="base_laser" type="fixed">
+	<joint name="base_laser_joint" type="fixed">
 		<parent link="base_link"/>
-		<child link="laser"/>
-		<origin xyz="-0.115 0 ${base_z_size}" rpy="0 0 ${M_PI}"/>
+		<child link="laser_link"/>
+		<origin xyz="0.10 0 ${base_z_size+0.015}" rpy="0 0 0"/>
 		<axis xyz="0 1 0"/>
 	</joint>

Commit message: Added namespace/prefix and twist mux

File: marrtino_description/urdf/marrtino_robot.xacro (robot description, xacro)
@@ -4,18 +4,11 @@
 	xmlns:controller="http://playerstage.sourceforge.net/gazebo/xmlschema/#controller"
 	xmlns:interface="http://playerstage.sourceforge.net/gazebo/xmlschema/#interface"
-	name="robot_xacro">
+	name="marrtino">
 	<xacro:include filename="$(find marrtino_description)/urdf/marrtino_robot.gazebo"/>
-    	<xacro:property name="M_PI" value="3.14159265359"/>
+  <xacro:property name="M_PI" value="3.14159265359"/>
 	<!-- Box Properties -->
 	<xacro:property name="base_x_size" value="0.28"/>
 	<xacro:property name="base_y_size" value="0.37"/>
 	<xacro:property name="base_z_size" value="0.21"/>
-  <!-- Wheel Mounting Positions -->
-	<!--
-	<xacro:property name="wheel_radius" value="0.07"/>
-  <xacro:property name="wheel_lenght" value="0.03"/>
-  <xacro:property name="castor_radius" value="0.03"/>
-  <xacro:property name="castor_length" value="0.015"/>
-  -->
 	<!-- Wheel Properties -->
 	<xacro:property name="wheel_radius" value="0.07"/>
@@ -156,22 +149,4 @@
 		<xacro:cylinder_inertia m="0.25" r="${castor_radius}" h="${castor_length}" />
 	</link>
-	<!-- Hokuyo Laser -->
-	<!--
-	<link name="laser_link" >
-		<visual>
-			<origin xyz="0 0 0" rpy="0 0 0"/>
-			<geometry>
-				<mesh filename="package://marrtino_description/meshes/hokuyo.dae"/>
-			</geometry>
-		</visual>
-		<collision>
-			<origin rpy="0 0 0" xyz="0 0 0"/>
-			<geometry>
-				<box size="0.1 0.1 0.1"/>
-			</geometry>
-		</collision>
-		<xacro:box_inertia m="0.05" x="0.1" y="0.1" z="0.1" />
-	</link>
--->
 	<link name="laser_link" >
 		<visual>

Commit message: Switch to prefix in front of tf (tf_prefix is deprecated)

File: marrtino_description/urdf/marrtino_robot.xacro (robot description, xacro)
@@ -5,4 +5,5 @@
 	xmlns:interface="http://playerstage.sourceforge.net/gazebo/xmlschema/#interface"
 	name="marrtino">
+	<xacro:arg name="prefix" default="marrtino_"/>
 	<xacro:include filename="$(find marrtino_description)/urdf/marrtino_robot.gazebo"/>
   <xacro:property name="M_PI" value="3.14159265359"/>
@@ -48,6 +49,6 @@
 	</xacro:macro>
 <!-- ..........................................Links definitions .....................................................-->
-	<link name="base_footprint"/>
-	<link name="base_link">
+	<link name="$(arg prefix)base_footprint"/>
+	<link name="$(arg prefix)base_link">
 		<visual>
 			<geometry>
@@ -67,5 +68,5 @@
 		<xacro:box_inertia m="5" x="${base_x_size}" y="${base_y_size}" z="${base_z_size}"/>
 	</link>
-	<link name="left_wheel_link">
+	<link name="$(arg prefix)left_wheel_link">
 		<visual>
 			<geometry>
@@ -85,5 +86,5 @@
 		<xacro:cylinder_inertia m="0.5" r="${wheel_radius}" h="${wheel_lenght}" />
 	</link>
-	<link name="right_wheel_link">
+	<link name="$(arg prefix)right_wheel_link">
 		<visual>
 			<geometry>
@@ -103,5 +104,5 @@
 		<xacro:cylinder_inertia m="0.5" r="${wheel_radius}" h="${wheel_lenght}" />
 	</link>
-	<link name="block" type="fixed">
+	<link name="$(arg prefix)block" type="fixed">
 		<visual>
 			<geometry>
@@ -121,5 +122,5 @@
 		<xacro:box_inertia m="0.05" x="0.03" y="0.03" z="0.05" />
 	</link>
-	<link name="castor_link">
+	<link name="$(arg prefix)castor_link">
 		<visual>
 			<geometry>
@@ -149,5 +150,5 @@
 		<xacro:cylinder_inertia m="0.25" r="${castor_radius}" h="${castor_length}" />
 	</link>
-	<link name="laser_link" >
+	<link name="$(arg prefix)laser_link" >
 		<visual>
 			<origin xyz="0 0 0" rpy="0 0 0"/>
@@ -168,38 +169,38 @@
 	</link>
 <!-- ..........................................Joints definitions .....................................................-->
-	<joint name="left_wheel_joint" type="continuous">
-		<parent link="base_link" />
-		<child link="left_wheel_link" />
+	<joint name="$(arg prefix)left_wheel_joint" type="continuous">
+		<parent link="$(arg prefix)base_link" />
+		<child link="$(arg prefix)left_wheel_link" />
 		<origin xyz="0.10 0.20 -0.03" rpy="0 0 0"/>
 		<axis xyz="0 1 0" />
 	</joint>
-	<joint name="right_wheel_joint" type="continuous">
-		<parent link="base_link" />
-		<child link="right_wheel_link" />
+	<joint name="$(arg prefix)right_wheel_joint" type="continuous">
+		<parent link="$(arg prefix)base_link" />
+		<child link="$(arg prefix)right_wheel_link" />
 		<origin xyz="0.10 -0.20 -0.03" rpy="0 0 0"/>-->
 		<axis xyz="0 1 0" />
 	</joint>
-	<joint name="castor_joint" type="fixed">
-		<parent link="block" />
-		<child link="castor_link" />
+	<joint name="$(arg prefix)castor_joint" type="fixed">
+		<parent link="$(arg prefix)block" />
+		<child link="$(arg prefix)castor_link" />
 		<origin xyz="0 0 -0.065" rpy="0 0 0"/>-->
 		<axis xyz="0 1 0" />
 	</joint>
-	<joint name="block_to_base_joint" type="fixed">
-		<parent link="base_link" />
-		<child link="block" />
+	<joint name="$(arg prefix)block_to_base_joint" type="fixed">
+		<parent link="$(arg prefix)base_link" />
+		<child link="$(arg prefix)block" />
 		<origin xyz="-0.085 0.0 0.0" rpy="0 0 0"/>
 		<axis xyz="0 1 0" />
 	</joint>
-  <joint name="base_footprint_joint" type="fixed">
-		<parent link="base_footprint" />
-		<child link="base_link" />
+  <joint name="$(arg prefix)base_footprint_joint" type="fixed">
+		<parent link="$(arg prefix)base_footprint" />
+		<child link="$(arg prefix)base_link" />
 		<origin xyz="0.0 0.0 ${wheel_radius + 0.03}" rpy="0 0 0"/>
 		<axis xyz="0 1 0" />
 	</joint>
 	<!--  Laser joint -->
-	<joint name="base_laser_joint" type="fixed">
-		<parent link="base_link"/>
-		<child link="laser_link"/>
+	<joint name="$(arg prefix)base_laser_joint" type="fixed">
+		<parent link="$(arg prefix)base_link"/>
+		<child link="$(arg prefix)laser_link"/>
 		<origin xyz="0.10 0 ${base_z_size+0.015}" rpy="0 0 0"/>
 		<axis xyz="0 1 0"/>

Commit message: Modified caster wheel and simulation fix

File: marrtino_description/urdf/marrtino_robot.xacro (robot description, xacro)
@@ -16,5 +16,4 @@
   <xacro:property name="wheel_lenght" value="0.03"/>
   <xacro:property name="castor_radius" value="0.03"/>
-  <xacro:property name="castor_length" value="0.015"/>
 	<xacro:macro name="default_inertial" params = "mass">
 		<inertial>
@@ -51,4 +50,5 @@
 	<link name="$(arg prefix)base_footprint"/>
 	<link name="$(arg prefix)base_link">
+		<xacro:box_inertia m="3" x="${base_x_size}" y="${base_y_size}" z="${base_z_size}"/>
 		<visual>
 			<geometry>
@@ -66,75 +66,18 @@
 			<origin xyz="0 0 ${base_z_size/2}" rpy = "0 0 0" />
 		</collision>
-		<xacro:box_inertia m="5" x="${base_x_size}" y="${base_y_size}" z="${base_z_size}"/>
-	</link>
-	<link name="$(arg prefix)left_wheel_link">
-		<visual>
-			<geometry>
-				<cylinder length="${wheel_lenght}" radius="${wheel_radius}"/>
-			</geometry>
-			<origin xyz="0 0 0" rpy="${M_PI/2} 0 0"/>
-			<material name="black">
-				<color rgba="0 0 0 1"/>
-			</material>
-		</visual>
-		<collision>
-			<geometry>
-				<cylinder length="${wheel_lenght}" radius="${wheel_radius}"/>
-			</geometry>
-			<origin xyz="0 0 0" rpy="${M_PI/2} 0 0"/>
-		</collision>
-		<xacro:cylinder_inertia m="0.5" r="${wheel_radius}" h="${wheel_lenght}" />
-	</link>
-	<link name="$(arg prefix)right_wheel_link">
-		<visual>
-			<geometry>
-				<cylinder length="${wheel_lenght}" radius="${wheel_radius}"/>
-			</geometry>
-			<origin xyz="0 0 0" rpy="${M_PI/2} 0 0"/>
-			<material name="black">
-				<color rgba="0 0 0 1"/>
-			</material>
-		</visual>
-		<collision>
-			<geometry>
-				<cylinder length="${wheel_lenght}" radius="${wheel_radius}"/>
-			</geometry>
-			<origin xyz="0 0 0" rpy="${M_PI/2} 0 0"/>
-		</collision>
-		<xacro:cylinder_inertia m="0.5" r="${wheel_radius}" h="${wheel_lenght}" />
-	</link>
-	<link name="$(arg prefix)block" type="fixed">
-		<visual>
-			<geometry>
-				<box size="0.03 0.03 0.05"/>
-			</geometry>
-			<origin xyz="0 0 -0.025" rpy = "0 0 0"/>
-			<material name="red">
-				<color rgba="1 0 0 1"/>
-			</material>
-		</visual>
-		<collision>
-			<geometry>
-				<box size="0.03 0.03 0.05"/>
-			</geometry>
-			<origin xyz="0 0 -0.05" rpy = "0 0 0"/>
-		</collision>
-		<xacro:box_inertia m="0.05" x="0.03" y="0.03" z="0.05" />
-	</link>
-	<link name="$(arg prefix)castor_link">
-		<visual>
-			<geometry>
-				<cylinder length="${castor_length}" radius="${castor_radius}"/>
-			</geometry>
-			<origin rpy="${M_PI/2} 0 0" xyz="0 0 0"/>
-			<material name="black">
-				<color rgba="0 0 0 1"/>
-			</material>
-		</visual>
-		<collision>
-			<geometry>
-				<cylinder length="${castor_length}" radius="${castor_radius}"/>
-			</geometry>
-			<origin rpy="${M_PI/2} 0 0" xyz="0 0 0"/>
+		<visual>
+			<geometry>
+				<sphere radius="${castor_radius}"/>
+			</geometry>
+			<origin rpy="0 0 0" xyz="-0.085 0 -0.07"/>
+			<material name="black">
+				<color rgba="0 0 0 1"/>
+			</material>
+		</visual>
+		<collision>
+			<geometry>
+				<sphere radius="${castor_radius}"/>
+			</geometry>
+			<origin rpy="0 0 0" xyz="-0.085 0 -0.07"/>
 			<surface>
         <friction>
@@ -148,6 +91,61 @@
 			</surface>
 		</collision>
-		<xacro:cylinder_inertia m="0.25" r="${castor_radius}" h="${castor_length}" />
-	</link>
+	</link>
+	<link name="$(arg prefix)left_wheel_link">
+		<visual>
+			<geometry>
+				<cylinder length="${wheel_lenght}" radius="${wheel_radius}"/>
+			</geometry>
+			<origin xyz="0 0 0" rpy="${M_PI/2} 0 0"/>
+			<material name="black">
+				<color rgba="0 0 0 1"/>
+			</material>
+		</visual>
+		<collision>
+			<geometry>
+				<cylinder length="${wheel_lenght}" radius="${wheel_radius}"/>
+			</geometry>
+			<origin xyz="0 0 0" rpy="${M_PI/2} 0 0"/>
+		</collision>
+		<xacro:cylinder_inertia m="0.3" r="${wheel_radius}" h="${wheel_lenght}" />
+	</link>
+	<link name="$(arg prefix)right_wheel_link">
+		<visual>
+			<geometry>
+				<cylinder length="${wheel_lenght}" radius="${wheel_radius}"/>
+			</geometry>
+			<origin xyz="0 0 0" rpy="${M_PI/2} 0 0"/>
+			<material name="black">
+				<color rgba="0 0 0 1"/>
+			</material>
+		</visual>
+		<collision>
+			<geometry>
+				<cylinder length="${wheel_lenght}" radius="${wheel_radius}"/>
+			</geometry>
+			<origin xyz="0 0 0" rpy="${M_PI/2} 0 0"/>
+		</collision>
+		<xacro:cylinder_inertia m="0.3" r="${wheel_radius}" h="${wheel_lenght}" />
+	</link>
+<!--
+	<link name="$(arg prefix)block" type="fixed">
+		<visual>
+			<geometry>
+				<box size="0.03 0.03 0.05"/>
+			</geometry>
+			<origin xyz="0 0 -0.025" rpy = "0 0 0"/>
+			<material name="red">
+				<color rgba="1 0 0 1"/>
+			</material>
+		</visual>
+		<collision>
+			<geometry>
+				<box size="0.03 0.03 0.05"/>
+			</geometry>
+			<origin xyz="0 0 -0.05" rpy = "0 0 0"/>
+		</collision>
+		<xacro:box_inertia m="0.05" x="0.03" y="0.03" z="0.05" />
+	</link>
+-->
 	<link name="$(arg prefix)laser_link" >
 		<visual>
@@ -181,8 +179,9 @@
 		<axis xyz="0 1 0" />
 	</joint>
+<!--
 	<joint name="$(arg prefix)castor_joint" type="fixed">
 		<parent link="$(arg prefix)block" />
 		<child link="$(arg prefix)castor_link" />
-		<origin xyz="0 0 -0.065" rpy="0 0 0"/>-->
+		<origin xyz="0 0 -0.065" rpy="0 0 0"/>
 		<axis xyz="0 1 0" />
 	</joint>
@@ -193,8 +192,9 @@
 		<axis xyz="0 1 0" />
 	</joint>
+-->
   <joint name="$(arg prefix)base_footprint_joint" type="fixed">
 		<parent link="$(arg prefix)base_footprint" />
 		<child link="$(arg prefix)base_link" />
-		<origin xyz="0.0 0.0 ${wheel_radius + 0.03}" rpy="0 0 0"/>
+		<origin xyz="0.0 0.0 ${wheel_radius + 0.04}" rpy="0 0 0"/>
 		<axis xyz="0 1 0" />
 	</joint>

Commit message: Added (old) diff_drive_plugin

File: marrtino_description/urdf/marrtino_robot.xacro (robot description, xacro)
@@ -7,5 +7,5 @@
 	<xacro:arg name="prefix" default="marrtino_"/>
 	<xacro:include filename="$(find marrtino_description)/urdf/marrtino_robot.gazebo"/>
-  <xacro:property name="M_PI" value="3.14159265359"/>
+	<xacro:property name="M_PI" value="3.1415926535897931"/>
 	<!-- Box Properties -->
 	<xacro:property name="base_x_size" value="0.28"/>
@@ -15,5 +15,5 @@
 	<xacro:property name="wheel_radius" value="0.07"/>
   <xacro:property name="wheel_lenght" value="0.03"/>
-  <xacro:property name="castor_radius" value="0.03"/>
+  <xacro:property name="castor_radius" value="0.02"/>
 	<xacro:macro name="default_inertial" params = "mass">
 		<inertial>
@@ -24,31 +24,26 @@
 	</xacro:macro>
 	<xacro:macro name="cylinder_inertia" params="m r h">
-		<inertial>
-		<mass value="${m}" />
 	     <inertia  ixx="${m*(3*r*r+h*h)/12}" ixy = "0" ixz = "0"
 	                  iyy="${m*(3*r*r+h*h)/12}" iyz = "0"
 	                  izz="${m*r*r/2}" />
-		</inertial>
 	</xacro:macro>
 	<xacro:macro name="box_inertia" params="m x y z">
-		<inertial>
-		<mass value="${m}" />
 	        <inertia  ixx="${m*(y*y+z*z)/12}" ixy = "0" ixz = "0"
 	                  iyy="${m*(x*x+z*z)/12}" iyz = "0"
 	                  izz="${m*(x*x+z*z)/12}" />
-				</inertial>
 	</xacro:macro>
 	<xacro:macro name="sphere_inertia" params="m r">
-		<inertial>
-		<mass value="${m}" />
-	        <inertia  ixx="${2*m*r*r/5}" ixy = "0" ixz = "0"
-	                  iyy="${2*m*r*r/5}" iyz = "0"
-	                  izz="${2*m*r*r/5}" />
-	  </inertial>
+	    <inertia  ixx="${2*m*r*r/5}" ixy = "0" ixz = "0"
+	              iyy="${2*m*r*r/5}" iyz = "0"
+	              izz="${2*m*r*r/5}" />
 	</xacro:macro>
 <!-- ..........................................Links definitions .....................................................-->
-	<link name="$(arg prefix)base_footprint"/>
+<link name="$(arg prefix)base_footprint" />
 	<link name="$(arg prefix)base_link">
-		<xacro:box_inertia m="3" x="${base_x_size}" y="${base_y_size}" z="${base_z_size}"/>
+		<inertial>
+			<origin xyz="0 0 ${base_z_size/2}" rpy = "0 0 0" />
+			<mass value="5" />
+			<xacro:box_inertia m="5" x="${base_x_size}" y="${base_y_size}" z="${base_z_size}"/>
+		</inertial>
 		<visual>
 			<geometry>
@@ -62,5 +57,5 @@
 		<collision>
 			<geometry>
-				<box size="${base_x_size} ${base_y_size} ${base_z_size}"/> <!--<box size="0.36 0.44 0.21"/>-->
+				<box size="${base_x_size} ${base_y_size} ${base_z_size}"/>
 			</geometry>
 			<origin xyz="0 0 ${base_z_size/2}" rpy = "0 0 0" />
@@ -68,26 +63,16 @@
 		<visual>
 			<geometry>
+				<sphere radius="${castor_radius}"/> <!--length="0.03-->
+			</geometry>
+			<origin xyz="-0.10 0 -0.06" rpy="${M_PI/2} 0 0"/>
+			<material name="black">
+				<color rgba="0 0 0 1"/>
+			</material>
+		</visual>
+		<collision>
+			<geometry>
 				<sphere radius="${castor_radius}"/>
 			</geometry>
-			<origin rpy="0 0 0" xyz="-0.085 0 -0.07"/>
-			<material name="black">
-				<color rgba="0 0 0 1"/>
-			</material>
-		</visual>
-		<collision>
-			<geometry>
-				<sphere radius="${castor_radius}"/>
-			</geometry>
-			<origin rpy="0 0 0" xyz="-0.085 0 -0.07"/>
-			<surface>
-        <friction>
-          <ode>
-            <mu>0</mu>
-            <mu2>0</mu2>
-            <slip1>1.0</slip1>
-            <slip2>1.0</slip2>
-          </ode>
-        </friction>
-			</surface>
+			<origin xyz="-0.10 0 -0.06" rpy="${M_PI/2} 0 0"/>
 		</collision>
 	</link>
@@ -108,5 +93,9 @@
 			<origin xyz="0 0 0" rpy="${M_PI/2} 0 0"/>
 		</collision>
-		<xacro:cylinder_inertia m="0.3" r="${wheel_radius}" h="${wheel_lenght}" />
+		<inertial>
+			<origin xyz="0 0 0" rpy = "${M_PI/2} 0 0" />
+			<mass value="1" />
+			<xacro:cylinder_inertia m="1" r="${wheel_radius}" h="${wheel_lenght}" />
+		</inertial>
 	</link>
 	<link name="$(arg prefix)right_wheel_link">
@@ -126,5 +115,9 @@
 			<origin xyz="0 0 0" rpy="${M_PI/2} 0 0"/>
 		</collision>
-		<xacro:cylinder_inertia m="0.3" r="${wheel_radius}" h="${wheel_lenght}" />
+		<inertial>
+			<origin xyz="0 0 0" rpy = "${M_PI/2} 0 0" />
+			<mass value="1" />
+			<xacro:cylinder_inertia m="1" r="${wheel_radius}" h="${wheel_lenght}" />
+		</inertial>
 	</link>
 <!--
@@ -164,5 +157,9 @@
 			</geometry>
 		</collision>
-		<xacro:cylinder_inertia m="0.05" r="0.04" h="0.03" />
+		<inertial>
+			<origin xyz="0 0 0" rpy = "0 0 0" />
+			<mass value="0.1" />
+			<xacro:cylinder_inertia m="0.1" r="0.04" h="0.03" />
+		</inertial>
 	</link>
 <!-- ..........................................Joints definitions .....................................................-->
@@ -170,12 +167,14 @@
 		<parent link="$(arg prefix)base_link" />
 		<child link="$(arg prefix)left_wheel_link" />
-		<origin xyz="0.10 0.20 -0.03" rpy="0 0 0"/>
-		<axis xyz="0 1 0" />
+		<origin xyz="0.10 0.20 -0.01" rpy="0 0 0"/>
+		<axis xyz="0 1 0" />
+		<joint_properties damping="0.0" friction="0.0"/>
 	</joint>
 	<joint name="$(arg prefix)right_wheel_joint" type="continuous">
 		<parent link="$(arg prefix)base_link" />
 		<child link="$(arg prefix)right_wheel_link" />
-		<origin xyz="0.10 -0.20 -0.03" rpy="0 0 0"/>-->
-		<axis xyz="0 1 0" />
+		<origin xyz="0.10 -0.20 -0.01" rpy="0 0 0"/>
+		<axis xyz="0 1 0" />
+		<joint_properties damping="0.0" friction="0.0"/>
 	</joint>
 <!--
