Commit message: Minor improvements

File: marrtino_description/urdf/marrtino_robot.xacro (robot description, xacro)
@@ -145,5 +145,5 @@
 			<origin xyz="0 0 0" rpy="0 0 0"/>
 			<geometry>
-				<cylinder length="0.03" radius="0.04"/>
+				<cylinder length="0.04" radius="0.035"/>
 			</geometry>
 			<material name="black">
@@ -154,5 +154,5 @@
 			<origin rpy="0 0 0" xyz="0 0 0"/>
 			<geometry>
-				<cylinder length="0.03" radius="0.04"/>
+				<cylinder length="0.04" radius="0.035"/>
 			</geometry>
 		</collision>
@@ -160,5 +160,5 @@
 			<origin xyz="0 0 0" rpy = "0 0 0" />
 			<mass value="0.1" />
-			<xacro:cylinder_inertia m="0.1" r="0.04" h="0.03" />
+			<xacro:cylinder_inertia m="0.1" r="0.035" h="0.04" />
 		</inertial>
 	</link>
@@ -167,5 +167,5 @@
 		<parent link="$(arg prefix)base_link" />
 		<child link="$(arg prefix)left_wheel_link" />
-		<origin xyz="0.10 0.20 -0.01" rpy="0 0 0"/>
+		<origin xyz="0.09 0.21 -0.015" rpy="0 0 0"/>
 		<axis xyz="0 1 0" />
 		<joint_properties damping="0.0" friction="0.0"/>
@@ -174,5 +174,5 @@
 		<parent link="$(arg prefix)base_link" />
 		<child link="$(arg prefix)right_wheel_link" />
-		<origin xyz="0.10 -0.20 -0.01" rpy="0 0 0"/>
+		<origin xyz="0.09 -0.21 -0.015" rpy="0 0 0"/>
 		<axis xyz="0 1 0" />
 		<joint_properties damping="0.0" friction="0.0"/>

Commit message: Added basket

File: marrtino_description/urdf/marrtino_robot.xacro (robot description, xacro)
@@ -16,10 +16,7 @@
   <xacro:property name="wheel_lenght" value="0.03"/>
   <xacro:property name="castor_radius" value="0.02"/>
-	<xacro:macro name="default_inertial" params = "mass">
-		<inertial>
-			<mass value="${mass}" />
+	<xacro:macro name="default_inertia" params = "m">
 			<inertia ixx="1.0" ixy = "0.0" ixz = "0.0"
 				 iyy="1.0" iyz = "0.0" izz = "1.0" />
-		</inertial>
 	</xacro:macro>
 	<xacro:macro name="cylinder_inertia" params="m r h">
@@ -121,11 +118,10 @@
 		</inertial>
 	</link>
-<!--
-	<link name="$(arg prefix)block" type="fixed">
+	<link name="$(arg prefix)basket">
 		<visual>
 			<geometry>
-				<box size="0.03 0.03 0.05"/>
+				<mesh filename="package://marrtino_description/meshes/basket.stl" />
 			</geometry>
-			<origin xyz="0 0 -0.025" rpy = "0 0 0"/>
+			<origin xyz="0 0 0" rpy = "0 0 ${M_PI/2}"/>
 			<material name="red">
 				<color rgba="1 0 0 1"/>
@@ -134,11 +130,9 @@
 		<collision>
 			<geometry>
-				<box size="0.03 0.03 0.05"/>
+				<mesh filename="package://marrtino_description/meshes/basket.stl" />
 			</geometry>
-			<origin xyz="0 0 -0.05" rpy = "0 0 0"/>
+			<origin xyz="0 0 0" rpy = "0 0 ${M_PI/2}"/>
 		</collision>
-		<xacro:box_inertia m="0.05" x="0.03" y="0.03" z="0.05" />
 	</link>
--->
 	<link name="$(arg prefix)laser_link" >
 		<visual>
@@ -178,18 +172,9 @@
 		<joint_properties damping="0.0" friction="0.0"/>
 	</joint>
-<!--
-	<joint name="$(arg prefix)castor_joint" type="fixed">
-		<parent link="$(arg prefix)block" />
-		<child link="$(arg prefix)castor_link" />
-		<origin xyz="0 0 -0.065" rpy="0 0 0"/>
-		<axis xyz="0 1 0" />
+	<joint name="$(arg prefix)basket_to_base_joint" type="fixed">
+		<parent link="$(arg prefix)base_link" />
+		<child link="$(arg prefix)basket" />
+		<origin xyz="0.0 0.0 ${base_z_size+0.40}" rpy="0 0 0"/>
 	</joint>
-	<joint name="$(arg prefix)block_to_base_joint" type="fixed">
-		<parent link="$(arg prefix)base_link" />
-		<child link="$(arg prefix)block" />
-		<origin xyz="-0.085 0.0 0.0" rpy="0 0 0"/>
-		<axis xyz="0 1 0" />
-	</joint>
--->
   <joint name="$(arg prefix)base_footprint_joint" type="fixed">
 		<parent link="$(arg prefix)base_footprint" />

Commit message: Fix formatting and remove map files

File: marrtino_description/urdf/marrtino_robot.xacro (robot description, xacro)
@@ -1,192 +1,192 @@
 <?xml version="1.0"?>
 <robot  xmlns:xacro= "http://www.ros.org/wiki/xacro"
-	xmlns:sensor="http://playerstage.sourceforge.net/gazebo/xmlschema/#sensor"
-	xmlns:controller="http://playerstage.sourceforge.net/gazebo/xmlschema/#controller"
-	xmlns:interface="http://playerstage.sourceforge.net/gazebo/xmlschema/#interface"
-	name="marrtino">
-	<xacro:arg name="prefix" default="marrtino_"/>
-	<xacro:include filename="$(find marrtino_description)/urdf/marrtino_robot.gazebo"/>
-	<xacro:property name="M_PI" value="3.1415926535897931"/>
-	<!-- Box Properties -->
-	<xacro:property name="base_x_size" value="0.28"/>
-	<xacro:property name="base_y_size" value="0.37"/>
-	<xacro:property name="base_z_size" value="0.21"/>
-	<!-- Wheel Properties -->
-	<xacro:property name="wheel_radius" value="0.07"/>
+    xmlns:sensor="http://playerstage.sourceforge.net/gazebo/xmlschema/#sensor"
+    xmlns:controller="http://playerstage.sourceforge.net/gazebo/xmlschema/#controller"
+    xmlns:interface="http://playerstage.sourceforge.net/gazebo/xmlschema/#interface"
+    name="marrtino">
+    <xacro:arg name="prefix" default="marrtino_"/>
+    <xacro:include filename="$(find marrtino_description)/urdf/marrtino_robot.gazebo"/>
+    <xacro:property name="M_PI" value="3.1415926535897931"/>
+    <!-- Box Properties -->
+    <xacro:property name="base_x_size" value="0.28"/>
+    <xacro:property name="base_y_size" value="0.37"/>
+    <xacro:property name="base_z_size" value="0.21"/>
+    <!-- Wheel Properties -->
+    <xacro:property name="wheel_radius" value="0.07"/>
   <xacro:property name="wheel_lenght" value="0.03"/>
   <xacro:property name="castor_radius" value="0.02"/>
-	<xacro:macro name="default_inertia" params = "m">
-			<inertia ixx="1.0" ixy = "0.0" ixz = "0.0"
-				 iyy="1.0" iyz = "0.0" izz = "1.0" />
-	</xacro:macro>
-	<xacro:macro name="cylinder_inertia" params="m r h">
-	     <inertia  ixx="${m*(3*r*r+h*h)/12}" ixy = "0" ixz = "0"
-	                  iyy="${m*(3*r*r+h*h)/12}" iyz = "0"
-	                  izz="${m*r*r/2}" />
-	</xacro:macro>
-	<xacro:macro name="box_inertia" params="m x y z">
-	        <inertia  ixx="${m*(y*y+z*z)/12}" ixy = "0" ixz = "0"
-	                  iyy="${m*(x*x+z*z)/12}" iyz = "0"
-	                  izz="${m*(x*x+z*z)/12}" />
-	</xacro:macro>
-	<xacro:macro name="sphere_inertia" params="m r">
-	    <inertia  ixx="${2*m*r*r/5}" ixy = "0" ixz = "0"
-	              iyy="${2*m*r*r/5}" iyz = "0"
-	              izz="${2*m*r*r/5}" />
-	</xacro:macro>
+    <xacro:macro name="default_inertia" params = "m">
+            <inertia ixx="1.0" ixy = "0.0" ixz = "0.0"
+                 iyy="1.0" iyz = "0.0" izz = "1.0" />
+    </xacro:macro>
+    <xacro:macro name="cylinder_inertia" params="m r h">
+         <inertia  ixx="${m*(3*r*r+h*h)/12}" ixy = "0" ixz = "0"
+                      iyy="${m*(3*r*r+h*h)/12}" iyz = "0"
+                      izz="${m*r*r/2}" />
+    </xacro:macro>
+    <xacro:macro name="box_inertia" params="m x y z">
+            <inertia  ixx="${m*(y*y+z*z)/12}" ixy = "0" ixz = "0"
+                      iyy="${m*(x*x+z*z)/12}" iyz = "0"
+                      izz="${m*(x*x+z*z)/12}" />
+    </xacro:macro>
+    <xacro:macro name="sphere_inertia" params="m r">
+        <inertia  ixx="${2*m*r*r/5}" ixy = "0" ixz = "0"
+                  iyy="${2*m*r*r/5}" iyz = "0"
+                  izz="${2*m*r*r/5}" />
+    </xacro:macro>
 <!-- ..........................................Links definitions .....................................................-->
 <link name="$(arg prefix)base_footprint" />
-	<link name="$(arg prefix)base_link">
-		<inertial>
-			<origin xyz="0 0 ${base_z_size/2}" rpy = "0 0 0" />
-			<mass value="5" />
-			<xacro:box_inertia m="5" x="${base_x_size}" y="${base_y_size}" z="${base_z_size}"/>
-		</inertial>
-		<visual>
-			<geometry>
-				<box size="${base_x_size} ${base_y_size} ${base_z_size}"/>
-			</geometry>
-			<origin xyz="0 0 ${base_z_size/2}" rpy = "0 0 0" />
-			<material name="red">
-				<color rgba="1 0 0 1"/>
-			</material>
-		</visual>
-		<collision>
-			<geometry>
-				<box size="${base_x_size} ${base_y_size} ${base_z_size}"/>
-			</geometry>
-			<origin xyz="0 0 ${base_z_size/2}" rpy = "0 0 0" />
-		</collision>
-		<visual>
-			<geometry>
-				<sphere radius="${castor_radius}"/> <!--length="0.03-->
-			</geometry>
-			<origin xyz="-0.10 0 -0.06" rpy="${M_PI/2} 0 0"/>
-			<material name="black">
-				<color rgba="0 0 0 1"/>
-			</material>
-		</visual>
-		<collision>
-			<geometry>
-				<sphere radius="${castor_radius}"/>
-			</geometry>
-			<origin xyz="-0.10 0 -0.06" rpy="${M_PI/2} 0 0"/>
-		</collision>
-	</link>
-	<link name="$(arg prefix)left_wheel_link">
-		<visual>
-			<geometry>
-				<cylinder length="${wheel_lenght}" radius="${wheel_radius}"/>
-			</geometry>
-			<origin xyz="0 0 0" rpy="${M_PI/2} 0 0"/>
-			<material name="black">
-				<color rgba="0 0 0 1"/>
-			</material>
-		</visual>
-		<collision>
-			<geometry>
-				<cylinder length="${wheel_lenght}" radius="${wheel_radius}"/>
-			</geometry>
-			<origin xyz="0 0 0" rpy="${M_PI/2} 0 0"/>
-		</collision>
-		<inertial>
-			<origin xyz="0 0 0" rpy = "${M_PI/2} 0 0" />
-			<mass value="1" />
-			<xacro:cylinder_inertia m="1" r="${wheel_radius}" h="${wheel_lenght}" />
-		</inertial>
-	</link>
-	<link name="$(arg prefix)right_wheel_link">
-		<visual>
-			<geometry>
-				<cylinder length="${wheel_lenght}" radius="${wheel_radius}"/>
-			</geometry>
-			<origin xyz="0 0 0" rpy="${M_PI/2} 0 0"/>
-			<material name="black">
-				<color rgba="0 0 0 1"/>
-			</material>
-		</visual>
-		<collision>
-			<geometry>
-				<cylinder length="${wheel_lenght}" radius="${wheel_radius}"/>
-			</geometry>
-			<origin xyz="0 0 0" rpy="${M_PI/2} 0 0"/>
-		</collision>
-		<inertial>
-			<origin xyz="0 0 0" rpy = "${M_PI/2} 0 0" />
-			<mass value="1" />
-			<xacro:cylinder_inertia m="1" r="${wheel_radius}" h="${wheel_lenght}" />
-		</inertial>
-	</link>
-	<link name="$(arg prefix)basket">
-		<visual>
-			<geometry>
-				<mesh filename="package://marrtino_description/meshes/basket.stl" />
-			</geometry>
-			<origin xyz="0 0 0" rpy = "0 0 ${M_PI/2}"/>
-			<material name="red">
-				<color rgba="1 0 0 1"/>
-			</material>
-		</visual>
-		<collision>
-			<geometry>
-				<mesh filename="package://marrtino_description/meshes/basket.stl" />
-			</geometry>
-			<origin xyz="0 0 0" rpy = "0 0 ${M_PI/2}"/>
-		</collision>
-	</link>
-	<link name="$(arg prefix)laser_link" >
-		<visual>
-			<origin xyz="0 0 0" rpy="0 0 0"/>
-			<geometry>
-				<cylinder length="0.04" radius="0.035"/>
-			</geometry>
-			<material name="black">
-				<color rgba="0 0 0 1"/>
-			</material>
-		</visual>
-		<collision>
-			<origin rpy="0 0 0" xyz="0 0 0"/>
-			<geometry>
-				<cylinder length="0.04" radius="0.035"/>
-			</geometry>
-		</collision>
-		<inertial>
-			<origin xyz="0 0 0" rpy = "0 0 0" />
-			<mass value="0.1" />
-			<xacro:cylinder_inertia m="0.1" r="0.035" h="0.04" />
-		</inertial>
-	</link>
+    <link name="$(arg prefix)base_link">
+        <inertial>
+            <origin xyz="0 0 ${base_z_size/2}" rpy = "0 0 0" />
+            <mass value="5" />
+            <xacro:box_inertia m="5" x="${base_x_size}" y="${base_y_size}" z="${base_z_size}"/>
+        </inertial>
+        <visual>
+            <geometry>
+                <box size="${base_x_size} ${base_y_size} ${base_z_size}"/>
+            </geometry>
+            <origin xyz="0 0 ${base_z_size/2}" rpy = "0 0 0" />
+            <material name="red">
+                <color rgba="1 0 0 1"/>
+            </material>
+        </visual>
+        <collision>
+            <geometry>
+                <box size="${base_x_size} ${base_y_size} ${base_z_size}"/>
+            </geometry>
+            <origin xyz="0 0 ${base_z_size/2}" rpy = "0 0 0" />
+        </collision>
+        <visual>
+            <geometry>
+                <sphere radius="${castor_radius}"/> <!--length="0.03-->
+            </geometry>
+            <origin xyz="-0.10 0 -0.06" rpy="${M_PI/2} 0 0"/>
+            <material name="black">
+                <color rgba="0 0 0 1"/>
+            </material>
+        </visual>
+        <collision>
+            <geometry>
+                <sphere radius="${castor_radius}"/>
+            </geometry>
+            <origin xyz="-0.10 0 -0.06" rpy="${M_PI/2} 0 0"/>
+        </collision>
+    </link>
+    <link name="$(arg prefix)left_wheel_link">
+        <visual>
+            <geometry>
+                <cylinder length="${wheel_lenght}" radius="${wheel_radius}"/>
+            </geometry>
+            <origin xyz="0 0 0" rpy="${M_PI/2} 0 0"/>
+            <material name="black">
+                <color rgba="0 0 0 1"/>
+            </material>
+        </visual>
+        <collision>
+            <geometry>
+                <cylinder length="${wheel_lenght}" radius="${wheel_radius}"/>
+            </geometry>
+            <origin xyz="0 0 0" rpy="${M_PI/2} 0 0"/>
+        </collision>
+        <inertial>
+            <origin xyz="0 0 0" rpy = "${M_PI/2} 0 0" />
+            <mass value="1" />
+            <xacro:cylinder_inertia m="1" r="${wheel_radius}" h="${wheel_lenght}" />
+        </inertial>
+    </link>
+    <link name="$(arg prefix)right_wheel_link">
+        <visual>
+            <geometry>
+                <cylinder length="${wheel_lenght}" radius="${wheel_radius}"/>
+            </geometry>
+            <origin xyz="0 0 0" rpy="${M_PI/2} 0 0"/>
+            <material name="black">
+                <color rgba="0 0 0 1"/>
+            </material>
+        </visual>
+        <collision>
+            <geometry>
+                <cylinder length="${wheel_lenght}" radius="${wheel_radius}"/>
+            </geometry>
+            <origin xyz="0 0 0" rpy="${M_PI/2} 0 0"/>
+        </collision>
+        <inertial>
+            <origin xyz="0 0 0" rpy = "${M_PI/2} 0 0" />
+            <mass value="1" />
+            <xacro:cylinder_inertia m="1" r="${wheel_radius}" h="${wheel_lenght}" />
+        </inertial>
+    </link>
+    <link name="$(arg prefix)basket">
+        <visual>
+            <geometry>
+                <mesh filename="package://marrtino_description/meshes/basket.stl" />
+            </geometry>
+            <origin xyz="0 0 0" rpy = "0 0 ${M_PI/2}"/>
+            <material name="red">
+                <color rgba="1 0 0 1"/>
+            </material>
+        </visual>
+        <collision>
+            <geometry>
+                <mesh filename="package://marrtino_description/meshes/basket.stl" />
+            </geometry>
+            <origin xyz="0 0 0" rpy = "0 0 ${M_PI/2}"/>
+        </collision>
+    </link>
+    <link name="$(arg prefix)laser_link" >
+        <visual>
+            <origin xyz="0 0 0" rpy="0 0 0"/>
+            <geometry>
+                <cylinder length="0.04" radius="0.035"/>
+            </geometry>
+            <material name="black">
+                <color rgba="0 0 0 1"/>
+            </material>
+        </visual>
+        <collision>
+            <origin rpy="0 0 0" xyz="0 0 0"/>
+            <geometry>
+                <cylinder length="0.04" radius="0.035"/>
+            </geometry>
+        </collision>
+        <inertial>
+            <origin xyz="0 0 0" rpy = "0 0 0" />
+            <mass value="0.1" />
+            <xacro:cylinder_inertia m="0.1" r="0.035" h="0.04" />
+        </inertial>
+    </link>
 <!-- ..........................................Joints definitions .....................................................-->
-	<joint name="$(arg prefix)left_wheel_joint" type="continuous">
-		<parent link="$(arg prefix)base_link" />
-		<child link="$(arg prefix)left_wheel_link" />
-		<origin xyz="0.09 0.21 -0.015" rpy="0 0 0"/>
-		<axis xyz="0 1 0" />
-		<joint_properties damping="0.0" friction="0.0"/>
-	</joint>
-	<joint name="$(arg prefix)right_wheel_joint" type="continuous">
-		<parent link="$(arg prefix)base_link" />
-		<child link="$(arg prefix)right_wheel_link" />
-		<origin xyz="0.09 -0.21 -0.015" rpy="0 0 0"/>
-		<axis xyz="0 1 0" />
-		<joint_properties damping="0.0" friction="0.0"/>
-	</joint>
-	<joint name="$(arg prefix)basket_to_base_joint" type="fixed">
-		<parent link="$(arg prefix)base_link" />
-		<child link="$(arg prefix)basket" />
-		<origin xyz="0.0 0.0 ${base_z_size+0.40}" rpy="0 0 0"/>
-	</joint>
+    <joint name="$(arg prefix)left_wheel_joint" type="continuous">
+        <parent link="$(arg prefix)base_link" />
+        <child link="$(arg prefix)left_wheel_link" />
+        <origin xyz="0.09 0.21 -0.015" rpy="0 0 0"/>
+        <axis xyz="0 1 0" />
+        <joint_properties damping="0.0" friction="0.0"/>
+    </joint>
+    <joint name="$(arg prefix)right_wheel_joint" type="continuous">
+        <parent link="$(arg prefix)base_link" />
+        <child link="$(arg prefix)right_wheel_link" />
+        <origin xyz="0.09 -0.21 -0.015" rpy="0 0 0"/>
+        <axis xyz="0 1 0" />
+        <joint_properties damping="0.0" friction="0.0"/>
+    </joint>
+    <joint name="$(arg prefix)basket_to_base_joint" type="fixed">
+        <parent link="$(arg prefix)base_link" />
+        <child link="$(arg prefix)basket" />
+        <origin xyz="0.0 0.0 ${base_z_size+0.40}" rpy="0 0 0"/>
+    </joint>
   <joint name="$(arg prefix)base_footprint_joint" type="fixed">
-		<parent link="$(arg prefix)base_footprint" />
-		<child link="$(arg prefix)base_link" />
-		<origin xyz="0.0 0.0 ${wheel_radius + 0.04}" rpy="0 0 0"/>
-		<axis xyz="0 1 0" />
-	</joint>
-	<!--  Laser joint -->
-	<joint name="$(arg prefix)base_laser_joint" type="fixed">
-		<parent link="$(arg prefix)base_link"/>
-		<child link="$(arg prefix)laser_link"/>
-		<origin xyz="0.10 0 ${base_z_size+0.015}" rpy="0 0 0"/>
-		<axis xyz="0 1 0"/>
-	</joint>
+        <parent link="$(arg prefix)base_footprint" />
+        <child link="$(arg prefix)base_link" />
+        <origin xyz="0.0 0.0 ${wheel_radius + 0.04}" rpy="0 0 0"/>
+        <axis xyz="0 1 0" />
+    </joint>
+    <!--  Laser joint -->
+    <joint name="$(arg prefix)base_laser_joint" type="fixed">
+        <parent link="$(arg prefix)base_link"/>
+        <child link="$(arg prefix)laser_link"/>
+        <origin xyz="0.10 0 ${base_z_size+0.015}" rpy="0 0 0"/>
+        <axis xyz="0 1 0"/>
+    </joint>
 </robot>

Commit message: Update friction coefficients and base_laser_joint roll orientation

File: marrtino_description/urdf/marrtino_robot.xacro (robot description, xacro)
@@ -187,5 +187,5 @@
         <parent link="$(arg prefix)base_link"/>
         <child link="$(arg prefix)laser_link"/>
-        <origin xyz="0.10 0 ${base_z_size+0.015}" rpy="0 0 0"/>
+        <origin xyz="0.10 0 ${base_z_size+0.015}" rpy="0.0001 0 0"/>
         <axis xyz="0 1 0"/>
     </joint>
